File: HVB/high-voltage-board/controller.sch (KiCad schematic (older format))
At the start: 30 parts, among them U1 STM32F413CGUx, U2 LD1117S33TR_SOT223

Commit message: working on schematic
Connections:
- net FAN_CTRL_0: no longer names the net of U1.11 (PA1)
- net FAN_CTRL_1: no longer names the net of U1.12 (PA2)
- net FAN_CTRL_2: no longer names the net of U1.15 (PA5)
- net FAN_CTRL_3: no longer names the net of U1.17 (PA7)
Changed lines of the file:
@@
 $Descr A4 11693 8268
 encoding utf-8
-Sheet 3 5
+Sheet 4 4
 Title ""
 Date ""
@@
 Wire Wire Line
 	2550 4800 2300 4800
-Text HLabel 4000 5200 2    50   Output ~ 0
-FAN_CTRL_0
-Text HLabel 4000 5300 2    50   Output ~ 0
-FAN_CTRL_1
-Text HLabel 4000 5600 2    50   Output ~ 0
-FAN_CTRL_2
-Text HLabel 4000 5800 2    50   Output ~ 0
-FAN_CTRL_3
 $Comp
 L Device:R_US R7
@@
 	4000 5900 3850 5900
 Wire Wire Line
-	3850 5800 4000 5800
-Wire Wire Line
 	4000 5700 3850 5700
 Wire Wire Line
-	3850 5600 4000 5600
-Wire Wire Line
 	4000 5500 3850 5500
 Wire Wire Line
 	3850 5400 4000 5400
 Wire Wire Line
-	4000 5300 3850 5300
-Wire Wire Line
-	3850 5200 4000 5200
-Wire Wire Line
 	4000 5100 3850 5100
