File: HVB/high-voltage-board/high-voltage-board.sch (KiCad schematic (older format))
At the start: 16 parts, among them J1 HECS, J16 Conn_01x23, J2 FANS, J3 NTCs, J4 Bender-LV, J6 HV+, J7 HV-, J8 HV+, U7 R-78E5.0-0.5

Commit message: changing connector pinout
Parts:
- removed J2: FANS, Connector_JST:JST_PH_B4B-PH-K_1x04_P2.00mm_Vertical, symbol Connector_Generic:Conn_01x04
Connections:
- net CAN+: now also J16.16 (Pin_16)
- net CAN-: now also J16.15 (Pin_15)
- net SHDN_LOOP_OUT renamed DCDC_OUT
- net DCDC_OUT: no longer J16.15 (Pin_15), J16.23 (Pin_23)
Other:
- note removed: "Willem Hillier\nUVM AERO\n3/5/2019"
Changed lines of the file:
@@
 DC_DC_FAULT
 Text Label 8700 3250 2    50   ~ 0
-SHDN_LOOP_OUT
-Wire Wire Line
-	1100 4500 1450 4500
-Text Label 1450 4500 2    50   ~ 0
-FANOUT0
-Wire Wire Line
-	1100 4600 1450 4600
-Text Label 1450 4600 2    50   ~ 0
-FANOUT0
-$Comp
-L power:+12V #PWR?
-U 1 1 5C8304FF
-P 1150 4250
-AR Path="/5C8304FF" Ref="#PWR?"  Part="1"
-AR Path="/5C83278E/5C8304FF" Ref="#PWR0110"  Part="1"
-F 0 "#PWR?" H 1150 4100 50  0001 C CNN
-F 1 "+12V" H 1165 4423 50  0000 C CNN
-F 2 "" H 1150 4250 50  0001 C CNN
-F 3 "" H 1150 4250 50  0001 C CNN
-	1    1150 4250
-	-1   0    0    -1
-$EndComp
-Wire Wire Line
-	1150 4250 1150 4300
-Wire Wire Line
-	1150 4300 1100 4300
+DCDC_OUT
 $Comp
 L Connector_Generic:Conn_01x05 J?
@@
 	-1   0    0    -1
 $EndComp
-Text Label 1800 6150 2    50   ~ 0
-SHDN_LOOP_OUT
 Wire Wire Line
 	1050 6150 1800 6150
-Text Label 1800 6850 2    50   ~ 0
-SHDN_LOOP_OUT
-Wire Wire Line
-	1050 6850 1800 6850
-Text Label 1800 7650 2    50   ~ 0
-SHDN_LOOP_OUT
-Wire Wire Line
-	1050 7650 1800 7650
 Wire Wire Line
 	1050 7250 1400 7250
 Wire Wire Line
 	1050 7050 1400 7050
-Text Label 1800 6050 2    50   ~ 0
-SHDN_LOOP_OUT
 Wire Wire Line
 	1050 6050 1800 6050
-Text Label 1800 6750 2    50   ~ 0
-SHDN_LOOP_OUT
 Wire Wire Line
 	1150 5750 1150 5850
@@
 Wire Wire Line
 	10325 5575 10325 5625
-Text Notes 8800 7050 0    100  ~ 0
-Willem Hillier\nUVM AERO\n3/5/2019
-$Comp
-L Connector_Generic:Conn_01x04 J2
-U 1 1 5CA58654
-P 900 4500
-F 0 "J2" H 820 4075 50  0000 C CNN
-F 1 "FANS" V 1000 4450 50  0000 C CNN
-F 2 "Connector_JST:JST_PH_B4B-PH-K_1x04_P2.00mm_Vertical" H 900 4500 50  0001 C CNN
-F 3 "~" H 900 4500 50  0001 C CNN
-	1    900  4500
-	-1   0    0    1
-$EndComp
 $Comp
 L Connector_Generic:Conn_01x04 J3
@@
 	-1   0    0    1
 $EndComp
-Wire Wire Line
-	1150 4300 1150 4400
-Wire Wire Line
-	1150 4400 1100 4400
-Connection ~ 1150 4300
 Wire Wire Line
 	2300 4300 2400 4300
@@
 Text Label 1400 7450 2    50   ~ 0
 TEMP_1
-Wire Wire Line
-	1050 6750 1800 6750
 Wire Wire Line
 	1050 5850 1150 5850
@@
 F8 "NTC2" I R 7950 2250 50
 $EndSheet
+Text Label 1800 6050 2    50   ~ 0
+DCDC_OUT
+Text Label 1800 6150 2    50   ~ 0
+DCDC_OUT
+Text Label 1800 6750 2    50   ~ 0
+DCDC_OUT
+Wire Wire Line
+	1050 6750 1800 6750
+Wire Wire Line
+	1050 6950 1400 6950
+Wire Wire Line
+	1050 6850 1400 6850
+Text Label 1400 6950 2    50   ~ 0
+CAN+
+Text Label 1400 6850 2    50   ~ 0
+CAN-
 $EndSCHEMATC
