File: HVB/high-voltage-board/controller.kicad_sch (KiCad schematic)
At the start: 24 parts, among them J12 Conn_01x02, Q3 DMN3404L, U4 LD1117S33TR_SOT223, U5 STM32F413CGUx, Y1 CSTME8M00

Commit message: updating layout and minor schem updates
Parts:
- C3: renamed from C?; footprint (none) -> Capacitor_SMD:C_0603_1608Metric_Pad1.08x0.95mm_HandSolder
- C7: renamed from C12; footprint (none) -> Capacitor_SMD:C_0603_1608Metric_Pad1.08x0.95mm_HandSolder
- J10: renamed from J?; footprint (none) -> Connector_PinHeader_1.27mm:PinHeader_2x07_P1.27mm_Vertical_SMD
- R11: renamed from R?; footprint (none) -> Resistor_SMD:R_0603_1608Metric_Pad0.98x0.95mm_HandSolder
- R13: renamed from R6; footprint (none) -> Resistor_SMD:R_0603_1608Metric_Pad0.98x0.95mm_HandSolder
- U1: renamed from U?; footprint SOIC127P600X175-8N -> AERO_Footprints:SOIC127P600X175-8N
- gave numbers to parts that had none: 1
Connections:
- net CAN_TX: now also U1.1 (TXD)
Changed lines of the file:
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@@
     (stroke (width 0) (type default) (color 0 0 0 0))
   )
-  (wire (pts (xy 203.2 132.08) (xy 208.28 132.08))
+  (wire (pts (xy 203.2 132.08) (xy 209.55 132.08))
     (stroke (width 0) (type default) (color 0 0 0 0))
   )
@@
   (symbol (lib_id "power:+3.3V") (at 217.17 109.22 0) (unit 1)
     (in_bom yes) (on_board yes) (fields_autoplaced)
-    (property "Reference" "#PWR?" (id 0) (at 217.17 113.03 0)
+    (property "Reference" "#PWR0116" (id 0) (at 217.17 113.03 0)
       (effects (font (size 1.27 1.27)) hide)
     )
@@
   (symbol (lib_id "power:GND") (at 217.17 116.84 0) (unit 1)
     (in_bom yes) (on_board yes) (fields_autoplaced)
-    (property "Reference" "#PWR?" (id 0) (at 217.17 123.19 0)
+    (property "Reference" "#PWR0115" (id 0) (at 217.17 123.19 0)
       (effects (font (size 1.27 1.27)) hide)
     )
@@
   (symbol (lib_id "Device:R") (at 214.63 135.89 0) (unit 1)
     (in_bom yes) (on_board yes)
-    (property "Reference" "R6" (id 0) (at 215.9 134.62 0)
+    (property "Reference" "R13" (id 0) (at 215.9 134.62 0)
       (effects (font (size 1.27 1.27)) (justify left))
     )
@@
       (effects (font (size 1.27 1.27)) (justify left))
     )
-    (property "Footprint" "" (id 2) (at 212.852 135.89 90)
+    (property "Footprint" "Resistor_SMD:R_0603_1608Metric_Pad0.98x0.95mm_HandSolder" (id 2) (at 212.852 135.89 90)
       (effects (font (size 1.27 1.27)) hide)
     )
@@
   (symbol (lib_id "Device:C") (at 207.01 113.03 0) (unit 1)
     (in_bom yes) (on_board yes)
-    (property "Reference" "C12" (id 0) (at 199.39 111.76 0)
+    (property "Reference" "C7" (id 0) (at 199.39 111.76 0)
       (effects (font (size 1.27 1.27)) (justify left))
     )
@@
       (effects (font (size 1.27 1.27)) (justify left))
     )
-    (property "Footprint" "" (id 2) (at 207.9752 116.84 0)
+    (property "Footprint" "Capacitor_SMD:C_0603_1608Metric_Pad1.08x0.95mm_HandSolder" (id 2) (at 207.9752 116.84 0)
       (effects (font (size 1.27 1.27)) hide)
     )
@@
   (symbol (lib_id "Device:C") (at 217.17 113.03 0) (unit 1)
     (in_bom yes) (on_board yes) (fields_autoplaced)
-    (property "Reference" "C?" (id 0) (at 220.98 111.7599 0)
+    (property "Reference" "C3" (id 0) (at 220.98 111.7599 0)
       (effects (font (size 1.27 1.27)) (justify left))
     )
@@
       (effects (font (size 1.27 1.27)) (justify left))
     )
-    (property "Footprint" "" (id 2) (at 218.1352 116.84 0)
+    (property "Footprint" "Capacitor_SMD:C_0603_1608Metric_Pad1.08x0.95mm_HandSolder" (id 2) (at 218.1352 116.84 0)
       (effects (font (size 1.27 1.27)) hide)
     )
@@
   (symbol (lib_id "power:+3.3V") (at 167.64 124.46 0) (unit 1)
     (in_bom yes) (on_board yes) (fields_autoplaced)
-    (property "Reference" "#PWR?" (id 0) (at 167.64 128.27 0)
+    (property "Reference" "#PWR0120" (id 0) (at 167.64 128.27 0)
       (effects (font (size 1.27 1.27)) hide)
     )
@@
   (symbol (lib_id "Connector_Generic:Conn_02x07_Odd_Even") (at 250.19 48.26 0) (unit 1)
     (in_bom yes) (on_board yes)
-    (property "Reference" "J?" (id 0) (at 251.46 33.02 0))
+    (property "Reference" "J10" (id 0) (at 251.46 33.02 0))
     (property "Value" "FTSH-107-01-F-DV-k" (id 1) (at 251.46 35.56 0))
-    (property "Footprint" "" (id 2) (at 250.19 48.26 0)
+    (property "Footprint" "Connector_PinHeader_1.27mm:PinHeader_2x07_P1.27mm_Vertical_SMD" (id 2) (at 250.19 48.26 0)
       (effects (font (size 1.27 1.27)) hide)
     )
@@
   (symbol (lib_id "AERO_Symbols:MAX33054EASA+T") (at 187.96 134.62 0) (mirror y) (unit 1)
     (in_bom yes) (on_board yes) (fields_autoplaced)
-    (property "Reference" "U?" (id 0) (at 187.96 116.84 0))
+    (property "Reference" "U1" (id 0) (at 187.96 116.84 0))
     (property "Value" "MAX33054EASA+T" (id 1) (at 187.96 119.38 0))
-    (property "Footprint" "SOIC127P600X175-8N" (id 2) (at 187.96 134.62 0)
+    (property "Footprint" "AERO_Footprints:SOIC127P600X175-8N" (id 2) (at 187.96 134.62 0)
       (effects (font (size 1.27 1.27)) (justify left bottom) hide)
     )
@@
   (symbol (lib_id "power:GND") (at 207.01 116.84 0) (unit 1)
     (in_bom yes) (on_board yes) (fields_autoplaced)
-    (property "Reference" "#PWR?" (id 0) (at 207.01 123.19 0)
+    (property "Reference" "#PWR0119" (id 0) (at 207.01 123.19 0)
       (effects (font (size 1.27 1.27)) hide)
     )
@@
   (symbol (lib_id "power:GND") (at 204.47 147.32 0) (unit 1)
     (in_bom yes) (on_board yes) (fields_autoplaced)
-    (property "Reference" "#PWR?" (id 0) (at 204.47 153.67 0)
+    (property "Reference" "#PWR0117" (id 0) (at 204.47 153.67 0)
       (effects (font (size 1.27 1.27)) hide)
     )
@@
   (symbol (lib_id "Device:R") (at 232.41 53.34 90) (unit 1)
     (in_bom yes) (on_board yes)
-    (property "Reference" "R?" (id 0) (at 232.41 50.8 90))
+    (property "Reference" "R11" (id 0) (at 232.41 50.8 90))
     (property "Value" "100" (id 1) (at 232.41 53.34 90))
-    (property "Footprint" "" (id 2) (at 232.41 55.118 90)
+    (property "Footprint" "Resistor_SMD:R_0603_1608Metric_Pad0.98x0.95mm_HandSolder" (id 2) (at 232.41 55.118 90)
       (effects (font (size 1.27 1.27)) hide)
     )
@@
   (symbol (lib_id "power:GND") (at 237.49 46.99 270) (unit 1)
     (in_bom yes) (on_board yes)
-    (property "Reference" "#PWR?" (id 0) (at 231.14 46.99 0)
+    (property "Reference" "#PWR0122" (id 0) (at 231.14 46.99 0)
       (effects (font (size 1.27 1.27)) hide)
     )
@@
   (symbol (lib_id "power:+3.3V") (at 207.01 109.22 0) (unit 1)
     (in_bom yes) (on_board yes) (fields_autoplaced)
-    (property "Reference" "#PWR?" (id 0) (at 207.01 113.03 0)
+    (property "Reference" "#PWR0118" (id 0) (at 207.01 113.03 0)
       (effects (font (size 1.27 1.27)) hide)
     )
@@
   (symbol (lib_id "Power_Protection:SP0502BAHT") (at 227.33 144.78 0) (unit 1)
     (in_bom yes) (on_board yes) (fields_autoplaced)
-    (property "Reference" "D?" (id 0) (at 233.68 143.5099 0)
+    (property "Reference" "D3" (id 0) (at 233.68 143.5099 0)
       (effects (font (size 1.27 1.27)) (justify left))
     )
@@
   (symbol (lib_id "power:GND") (at 172.72 147.32 0) (unit 1)
     (in_bom yes) (on_board yes) (fields_autoplaced)
-    (property "Reference" "#PWR?" (id 0) (at 172.72 153.67 0)
-      (effects (font (size 1.27 1.27)) hide)
-    )
+    (property "Reference" "#PWR0121" (id 0) (at 172.72 153.67 0)
+      (effects (font (size 1.27 1.27)) hide)
+    )

Commit message: finish layout ready for review
Parts:
- added JP1: SolderJumper_2_Bridged, Jumper:SolderJumper-2_P1.3mm_Bridged_RoundedPad1.0x1.5mm, symbol Jumper:SolderJumper_2_Bridged
Connections:
- net GND: now also C10.1, D3.3 (A), JP1.1 (A); no longer C10.2, U5.44 (BOOT0)
- net at U5.7 (NRST): now also C10.2; no longer C10.1
- net CAN_N renamed CAN-
- net CAN_P renamed CAN+
- new net: JP1.2 (B), U5.44 (BOOT0)
Other:
- moved on the sheet: C10, C13, Y1

Commit message: touching up layout and making gerbers
Parts:
- removed D1: BAT54GW, Diode_SMD:D_SOD-123, symbol Device:D_Schottky
Connections:
- net +12V: now also C9.1, U4.3 (VI)
- net +3V3: now also R7.2; no longer D2.2 (A)
- net GND: now also D2.1 (K); no longer R7.1
- new net: D2.2 (A), R7.1
Other:
- moved on the sheet: C12, C9, D2, R7, U4

Commit message: Addded comments
Other:
- note added: "DESD2CAN"
- note added: "DNP"
- note added: "Need to add TSV and/or flyback diodes to help w/ tranience"
Changed lines of the file:
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@@
     (stroke (width 0) (type default) (color 0 0 0 0))
+  )
+  (text "Need to add\nTSV and/or flyback diodes\nto help w/ tranience"
+    (at 35.56 56.515 0)
+    (effects (font (size 1.27 1.27) bold italic) (justify left bottom))
   )
   (text "G.Spearing\nFebruary 2022" (at 224.79 179.07 0)
@@
   (text "Fan Control" (at 144.78 18.415 0)
     (effects (font (size 1.27 1.27)) (justify left bottom))
+  )
+  (text "DESD2CAN" (at 235.585 150.495 0)
+    (effects (font (size 1.27 1.27) bold italic) (justify left bottom))
   )
   (text "PROGRAMMING" (at 256.54 30.48 180)
@@
     (effects (font (size 2.9972 2.9972)) (justify right bottom))
   )
+  (text "DNP" (at 219.71 135.255 0)
+    (effects (font (size 1.27 1.27) bold italic) (justify left bottom))
+  )
   (label "CAN_RX" (at 106.68 157.48 180)
