File: HVB/high-voltage-board/high-voltage-board.kicad_sch (KiCad schematic)
At the start: 18 parts, among them J1 Conn_01x23, J11 HV-, J2 HECS, J3 HV+, J4 HV-, J5 HV+, J6 HV-, J7 Conn_01x02, J8 HV+, J9 Bender-LV

Commit message: touching up layout and making gerbers
Other:
- note added: "Board Function: - CAN IN/OUT from RCB to DCB and Pack 1 - Vicor DC/DC - TSMP - BMS Current - STM32 (Precharge) - TSAL - IMD"
Changed lines of the file:
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@@
+    (effects (font (size 1.27 1.27)) (justify left bottom))
+  )
+  (text "Board Function: \n- CAN IN/OUT from RCB to DCB and Pack 1\n- Vicor DC/DC \n- TSMP\n- BMS Current\n- STM32 (Precharge)\n- TSAL\n- IMD"
+    (at 177.8 182.245 0)
     (effects (font (size 1.27 1.27)) (justify left bottom))
   )
@@
       (reference "C23") (unit 1) (value "4700uF") (footprint "Capacitor_THT:C_Radial_D18.0mm_H35.5mm_P7.50mm")
     )
-    (path "/00000000-0000-0000-0000-00005c8304a7/00000000-0000-0000-0000-000061903c93"
-      (reference "D1") (unit 1) (value "BAT54GW") (footprint "Diode_SMD:D_SOD-123")
-    )
     (path "/00000000-0000-0000-0000-00005c8304a7/00000000-0000-0000-0000-000061904301"

Commit message: Addded comments
Other:
- note added: "12v comes from DC/DC not GLV"
- note added: "Check IMD grounding requirments. May need to seperate ground points for testing insulation."
- note added: "GND to Frame"
- note added: "Goes to GLV MS then to RCB"
- note added: "Wrong footprint hits pcb edge"
Changed lines of the file:
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@@
     (effects (font (size 1.27 1.27)) (justify left bottom))
+  )
+  (text "12v comes from DC/DC not GLV" (at 132.715 170.815 0)
+    (effects (font (size 1.27 1.27) bold italic) (justify left bottom))
+  )
+  (text "Goes to GLV MS then to RCB" (at 34.925 136.525 0)
+    (effects (font (size 1.27 1.27) (thickness 0.254) bold italic) (justify left bottom))
   )
   (text "Vicor temperature sensor" (at 62.23 184.785 0)
@@
   (text "EMUS Current Sensor from BMS" (at 64.135 158.115 0)
     (effects (font (size 1.27 1.27)) (justify left bottom))
+  )
+  (text "GND to Frame\n" (at 40.005 158.75 0)
+    (effects (font (size 1.27 1.27) bold italic) (justify left bottom))
   )
   (text "CAN Goes to Pack 1\nand Dash" (at 32.385 131.445 0)
@@
     (effects (font (size 1.27 1.27)) (justify left bottom))
   )
+  (text "Check IMD grounding requirments. \nMay need to seperate ground points for testing insulation."
+    (at 21.59 125.73 0)
+    (effects (font (size 1.27 1.27) bold italic) (justify left bottom))
+  )
+  (text "Wrong footprint hits pcb edge" (at 19.05 182.245 90)
+    (effects (font (size 1.27 1.27) (thickness 0.254) bold italic) (justify left bottom))
+  )
   (label "HECS_AN1" (at 35.56 176.53 180)
