File: HVB/high-voltage-board/vicor.kicad_sch (KiCad schematic)
At the start: 18 parts, among them U7 Vicor_AERO, U8 LTV-817S, U9 TLP184

Commit message: working on layout
Updating traces for RCB and organizing HVB
Connections:
- net +5V renamed +3V3
Changed lines of the file:
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@@
-    (pin "1")
-  )
-  (symbol (lib_id "power:+5V") (at 149.86 90.17 0) (unit 1)
-    (in_bom yes) (on_board yes)
-    (property "Reference" "#PWR044" (id 0) (at 149.86 93.98 0)
-      (effects (font (size 1.27 1.27)) hide)
-    )
-    (property "Value" "+5V" (id 1) (at 150.241 85.7758 0))
-    (property "Footprint" "" (id 2) (at 149.86 90.17 0)
-      (effects (font (size 1.27 1.27)) hide)
-    )
-    (property "Datasheet" "" (id 3) (at 149.86 90.17 0)
-      (effects (font (size 1.27 1.27)) hide)
-    )
     (pin "1")
   )
@@
     (pin "9")
   )
+  (symbol (lib_id "power:+3.3V") (at 149.86 90.17 0) (unit 1)
+    (in_bom yes) (on_board yes) (fields_autoplaced)
+    (property "Reference" "#PWR0105" (id 0) (at 149.86 93.98 0)
+      (effects (font (size 1.27 1.27)) hide)
+    )
+    (property "Value" "+3.3V" (id 1) (at 149.86 86.5655 0))
+    (property "Footprint" "" (id 2) (at 149.86 90.17 0)
+      (effects (font (size 1.27 1.27)) hide)
+    )
+    (property "Datasheet" "" (id 3) (at 149.86 90.17 0)
+      (effects (font (size 1.27 1.27)) hide)
+    )
+    (pin "1")
+  )
 )

Commit message: almost done with layout
HV layout almost done. Tracing
Connections:
- net GND: now also U7.8 (-OUT); no longer U7.9 (-OUT)
- net at C22.1, L2.1, R20.2: now also U7.9 (+OUT); no longer U7.8 (+OUT)
Changed lines of the file:
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@@
     (pin "4")
     (pin "5")
+    (pin "9")
     (pin "8")
-    (pin "9")
   )
   (symbol (lib_id "power:+3.3V") (at 149.86 90.17 0) (unit 1)

Commit message: updating pcb size and layout
Parts:
- C19, C20, C21, C22, C23, C24: footprint Capacitor_THT:C_Radial_D8.0mm_H7.0mm_P3.50mm -> Capacitor_THT:C_Radial_D18.0mm_H35.5mm_P7.50mm
Changed lines of the file:
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@@
       (effects (font (size 1.27 1.27)) (justify left))
     )
-    (property "Footprint" "Capacitor_THT:C_Radial_D8.0mm_H7.0mm_P3.50mm" (id 2) (at 172.72 138.43 0)
+    (property "Footprint" "Capacitor_THT:C_Radial_D18.0mm_H35.5mm_P7.50mm" (id 2) (at 172.72 138.43 0)
       (effects (font (size 1.27 1.27)) hide)
     )
@@
       (effects (font (size 1.27 1.27)) (justify left))
     )
-    (property "Footprint" "Capacitor_THT:C_Radial_D8.0mm_H7.0mm_P3.50mm" (id 2) (at 104.14 142.24 0)
+    (property "Footprint" "Capacitor_THT:C_Radial_D18.0mm_H35.5mm_P7.50mm" (id 2) (at 104.14 142.24 0)
       (effects (font (size 1.27 1.27)) hide)
     )
@@
       (effects (font (size 1.27 1.27)) (justify left))
     )
-    (property "Footprint" "Capacitor_THT:C_Radial_D8.0mm_H7.0mm_P3.50mm" (id 2) (at 107.95 142.24 0)
+    (property "Footprint" "Capacitor_THT:C_Radial_D18.0mm_H35.5mm_P7.50mm" (id 2) (at 107.95 142.24 0)
       (effects (font (size 1.27 1.27)) hide)
     )
@@
       (effects (font (size 1.27 1.27)) (justify left))
     )
-    (property "Footprint" "Capacitor_THT:C_Radial_D8.0mm_H7.0mm_P3.50mm" (id 2) (at 111.76 142.24 0)
+    (property "Footprint" "Capacitor_THT:C_Radial_D18.0mm_H35.5mm_P7.50mm" (id 2) (at 111.76 142.24 0)
       (effects (font (size 1.27 1.27)) hide)
     )
@@
       (effects (font (size 1.27 1.27)) (justify left))
     )
-    (property "Footprint" "Capacitor_THT:C_Radial_D8.0mm_H7.0mm_P3.50mm" (id 2) (at 156.21 138.43 0)
+    (property "Footprint" "Capacitor_THT:C_Radial_D18.0mm_H35.5mm_P7.50mm" (id 2) (at 156.21 138.43 0)
       (effects (font (size 1.27 1.27)) hide)
     )
@@
       (effects (font (size 1.27 1.27)) (justify left))
     )
-    (property "Footprint" "Capacitor_THT:C_Radial_D8.0mm_H7.0mm_P3.50mm" (id 2) (at 177.8 138.43 0)
+    (property "Footprint" "Capacitor_THT:C_Radial_D18.0mm_H35.5mm_P7.50mm" (id 2) (at 177.8 138.43 0)
       (effects (font (size 1.27 1.27)) hide)
     )
@@
     (pin "4")
     (pin "5")
+    (pin "8")
     (pin "9")
-    (pin "8")
   )
   (symbol (lib_id "power:+3.3V") (at 149.86 90.17 0) (unit 1)

Commit message: Layout and Footprints update
Connections:
- net TRIM_HV renamed TRIM_EN
Changed lines of the file:
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@@
     (stroke (width 0) (type default) (color 0 0 0 0))
   )
-  (wire (pts (xy 113.03 41.91) (xy 128.27 41.91))
+  (wire (pts (xy 113.03 41.91) (xy 122.555 41.91))
     (stroke (width 0) (type default) (color 0 0 0 0))
   )
@@
     (effects (font (size 1.27 1.27)) (justify left bottom))
   )
-  (label "TRIM_HV" (at 128.27 41.91 180)
+  (label "TRIM_HV" (at 122.555 41.91 180)
     (effects (font (size 1.27 1.27)) (justify right bottom))
   )
@@
     (effects (font (size 1.27 1.27)) (justify right))
   )
+  (hierarchical_label "TRIM_EN" (shape input) (at 122.555 41.91 0)
+    (effects (font (size 1.27 1.27)) (justify left))
+  )
   (hierarchical_label "12V_OUT" (shape input) (at 182.88 135.89 0)

Commit message: Major Review and Part Update
updating footprints, component values, layouts
Parts:
- removed C20, C21: 0.68uF, Capacitor_THT:C_Radial_D18.0mm_H35.5mm_P7.50mm, symbol Device:C_Small
- removed C24: 4700uF, Capacitor_THT:C_Radial_D18.0mm_H35.5mm_P7.50mm, symbol Device:C_Small
- removed R16: 6.8k, Resistor_SMD:R_0603_1608Metric_Pad0.98x0.95mm_HandSolder, symbol Device:R_US
- added C2: 0.68uF, Capacitor_THT:C_Rect_L18.0mm_W8.0mm_P15.00mm_FKS3_FKP3, symbol Device:C_Small
- added R8: 300, Resistor_SMD:R_0603_1608Metric_Pad0.98x0.95mm_HandSolder, symbol Device:R
- C19: footprint Capacitor_THT:C_Radial_D18.0mm_H35.5mm_P7.50mm -> Capacitor_THT:C_Rect_L18.0mm_W8.0mm_P15.00mm_FKS3_FKP3
- L1: footprint Inductor_SMD:L_Murata_LQH55DN_5.7x5.0mm -> Inductor_SMD:L_1008_2520Metric_Pad1.43x2.20mm_HandSolder
- L2: footprint Inductor_SMD:L_Murata_LQH55DN_5.7x5.0mm -> Inductor_SMD:L_0805_2012Metric_Pad1.15x1.40mm_HandSolder
- R15, R20: value 1Ω -> 1
- RV1: value 50k -> 50k TC33x-2-503E; footprint Potentiometer_THT:Potentiometer_ACP_CA9-V10_Vertical -> Potentiometer_SMD:Potentiometer_Bourns_TC33X_Vertical
Connections:
- net HV-: now also RV1.1, C2.2
- net at RV1.2: now also R8.2
- net at C19.1, L1.2, R15.1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: now also C2.1
- net TRIM_EN: no longer names the net of RV1.3
- net TRIM_EN: no longer U7.2 (TR)
- new net TRIM_HV: R8.1, U7.2 (TR)
Other:
- note added: "FAULT_HV can only supply 4mA absolute max, hence the different optocoupler choice."
- note added: "HV Side is pulled high enternally, optoisolator turns on (with high signal) to pull en_hv low"
- note removed: "FAULT_HV can only supply 5mA absolute max, hence the different optocoupler choice."
- note removed: "Will probably switch back to half as many 4700uF caps."
- moved on the sheet: C22, C23, L2, R20

Commit message: Addded comments
Other:
- note added: "Change symbol footprint to show +/-"
- note added: "DC/DC out"
Changed lines of the file:
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@@
     (stroke (width 0) (type default) (color 0 0 0 0))
+  )
+  (text "DC/DC out" (at 189.865 136.525 0)
+    (effects (font (size 1.27 1.27) bold italic) (justify left bottom))
   )
   (text "Output Filtering" (at 162.56 124.46 0)
@@
     (effects (font (size 2.54 2.54)) (justify left bottom))
   )
+  (text "Change symbol footprint to show +/-" (at 189.865 146.685 0)
+    (effects (font (size 1.27 1.27) bold italic) (justify left bottom))
+  )
   (text "Pull high to disable" (at 152.4 74.93 0)
