File: RCB/rear-control-board/Controller.sch (KiCad schematic (older format))
At the start: 31 parts, among them U1 STM32F413CGUx, U2 LD1117S33TR_SOT223

Commit message: finish schematic, start layout
Parts:
- removed J? (x2): Conn_01x03, symbol Connector_Generic:Conn_01x03
- removed SW?: SW_Push, symbol Switch:SW_Push
- removed SW? (x2): SW_SPDT, symbol Switch:SW_SPDT
- removed SW?: SW_SPST, symbol Switch:SW_SPST
- C1, C10, C11, C12, C4, C5, C6, C7, C8, C9: renamed from C?; footprint (none) -> Capacitor_SMD:C_0603_1608Metric_Pad1.08x0.95mm_HandSolder
- C2, C3: footprint (none) -> Capacitor_SMD:C_0603_1608Metric_Pad1.08x0.95mm_HandSolder
- D1: footprint (none) -> Diode_SMD:D_SMB
- D2: footprint (none) -> LED_SMD:LED_0603_1608Metric_Pad1.05x0.95mm_HandSolder
- J6: renamed from J?; footprint (none) -> Connector_JST:JST_XH_B5B-XH-A_1x05_P2.50mm_Vertical
- R1: footprint (none) -> Resistor_SMD:R_0603_1608Metric_Pad0.98x0.95mm_HandSolder
- R2, R3, R4, R5, R6: renamed from R?; footprint (none) -> Resistor_SMD:R_0603_1608Metric_Pad0.98x0.95mm_HandSolder
- Y1: renamed from Y?; footprint (none) -> Crystal:Crystal_HC49-U_Vertical
- gave numbers to parts that had none: 1
Connections:
- net +3V3: now also U1.17 (PA7)
- net CAN_N: now also R6.2
- net CAN_RX_N: no longer U1.33 (PA12)
- net CAN_TX_P: no longer U1.32 (PA11)
Other:
- note removed: "Boot Pin Switches"
- note removed: "CAN"
- moved on the sheet: C12, R5, R6, U4
