File: RCB/rear-control-board/FET_OUTPUT.sch (KiCad schematic (older format))
At the start: 3 parts

Commit message: finish schematic, start layout
Parts:
- gave numbers to parts that had none: 3
Changed lines of the file:
@@
 $Descr A4 11693 8268
 encoding utf-8
-Sheet 4 6
+Sheet 4 5
 Title ""
 Date ""
@@
 $EndDescr
 $Comp
-L Transistor_FET:STB15N80K5 Q?
+L Transistor_FET:STB15N80K5 Q3
 U 1 1 61F4E7F1
 P 2200 2700
-F 0 "Q?" H 2400 2600 50  0000 L CNN
+F 0 "Q3" H 2400 2600 50  0000 L CNN
 F 1 "STB15N80K5" H 2350 2450 50  0000 L CNN
 F 2 "Package_TO_SOT_SMD:TO-263-2" H 2400 2625 50  0001 L CIN
@@
 $EndComp
 $Comp
-L power:GND #PWR?
+L power:GND #PWR0121
 U 1 1 61F4EF4B
 P 3450 3200
-F 0 "#PWR?" H 3450 2950 50  0001 C CNN
+F 0 "#PWR0121" H 3450 2950 50  0001 C CNN
 F 1 "GND" H 3455 3027 50  0000 C CNN
 F 2 "" H 3450 3200 50  0001 C CNN
@@
 $EndComp
 $Comp
-L Transistor_FET:STB15N80K5 Q?
+L Transistor_FET:STB15N80K5 Q4
 U 1 1 61F4F19F
 P 3350 2750
-F 0 "Q?" H 3550 2650 50  0000 L CNN
+F 0 "Q4" H 3550 2650 50  0000 L CNN
 F 1 "STB15N80K5" H 3550 2500 50  0000 L CNN
 F 2 "Package_TO_SOT_SMD:TO-263-2" H 3550 2675 50  0001 L CIN
@@
 $EndComp
 $Comp
-L Transistor_FET:STB15N80K5 Q?
+L Transistor_FET:STB15N80K5 Q5
 U 1 1 61F4FA3C
 P 4500 2750
-F 0 "Q?" H 4750 2650 50  0000 L CNN
+F 0 "Q5" H 4750 2650 50  0000 L CNN
 F 1 "STB15N80K5" H 4700 2500 50  0000 L CNN
 F 2 "Package_TO_SOT_SMD:TO-263-2" H 4700 2675 50  0001 L CIN
