File: RCB/rear-control-board/FAULT_LATCHER.sch (KiCad schematic (older format))
At the start: 8 parts, among them J4 Conn_01x02, J5 Conn_01x02, K2 G5V-2, K3 G5V-2, Q1 BSS84, Q2 2N7002

Commit message: working on layout
Changed lines of the file:
@@
 Wire Wire Line
 	5100 2650 5325 2650
-Text HLabel 3250 1750 0    50   Input ~ 0
+Text HLabel 3125 1750 0    50   Input ~ 0
 LOOP_IN
 Wire Wire Line
-	3250 1750 3500 1750
-Text HLabel 6250 1850 2    50   Output ~ 0
+	3125 1750 3500 1750
+Text HLabel 6500 1850 2    50   Output ~ 0
 LOOP_OUT
 Wire Wire Line
-	6250 1850 6000 1850
+	6500 1850 6000 1850
 Text HLabel 6150 2250 2    50   Input ~ 0
 IMD_FAULT_SIG
@@
 Text Label 4350 2650 0    50   ~ 0
 12V
+Text Label 3175 1750 0    50   ~ 0
+Loop_IN
+Text Label 6375 1850 2    50   ~ 0
+Loop_Out
 $EndSCHEMATC
