File: RCB/rear-control-board/FET_OUTPUT.kicad_sch (KiCad schematic)
At the start: 15 parts, among them U5 BV1HAL45EFJ, U6 BV1HAL45EFJ, U7 BV1HAL45EFJ

Commit message: Addded comments
Parts:
- added R?: 10k, symbol Device:R
Connections:
- net GND: now also R?.1
- new net Brake_out: R?.2
Other:
- note added: "*On startup, all 0v, then signal high, out is 12v, signal low, out is 8.44v"
- note added: "Add pulldown on all three output"
- note added: "All three only go down to 8.5v when signal is low"
- note added: "From STM32 3.3 High 0v low"
- note added: "NOTE: Pump is always on and does not need switching was removed and is now always on. Brake works fine and is in place. Fan was to high of a current draw for the BV1HAL45EFJ so is currently always on, in the future will find an apropriate load switch."
- note added: "Pulled to ground"
- note added: "Should be 50k"
- note added: "Should limit between 50-100uA"
Changed lines of the file:
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@@
+    (stroke (width 0) (type default) (color 0 0 0 0))
+  )
+  (wire (pts (xy 204.47 82.55) (xy 206.375 82.55))
     (stroke (width 0) (type default) (color 0 0 0 0))
   )
@@
     (stroke (width 0) (type default) (color 0 0 0 0))
   )
+  (wire (pts (xy 213.995 82.55) (xy 220.345 82.55))
+    (stroke (width 0) (type default) (color 0 0 0 0))
+  )
   (wire (pts (xy 113.03 66.04) (xy 113.03 69.215))
     (stroke (width 0) (type default) (color 0 0 0 0))
+  )
+  (text "Should be 50k\n" (at 144.145 88.265 0)
+    (effects (font (size 1.27 1.27) bold italic) (justify left bottom))
+  )
+  (text "Pulled to ground\n" (at 202.565 80.645 0)
+    (effects (font (size 1.27 1.27) bold italic) (justify left bottom))
+  )
+  (text "All three only go down to 8.5v when signal is low" (at 22.86 102.235 0)
+    (effects (font (size 1.27 1.27) bold italic) (justify left bottom))
+  )
+  (text "NOTE: Pump is always on and does not need switching was removed and is now always on.\nBrake works fine and is in place.\nFan was to high of a current draw for the BV1HAL45EFJ\nso is currently always on, in the future will find an apropriate load switch."
+    (at 34.925 131.445 0)
+    (effects (font (size 1.27 1.27) bold italic) (justify left bottom))
+  )
+  (text "Should limit between 50-100uA" (at 39.37 55.88 0)
+    (effects (font (size 1.27 1.27) bold italic) (justify left bottom))
   )
   (text "2.2mA current \nlimiting resistor " (at 45.974 60.96 0)
     (effects (font (size 1.27 1.27)) (justify left bottom))
   )
+  (text "Add pulldown on all three output\n" (at 95.885 31.75 0)
+    (effects (font (size 1.27 1.27) bold italic) (justify left bottom))
+  )
+  (text "*On startup, all 0v, then signal high, out is 12v, signal low, out is 8.44v"
+    (at 22.86 106.045 0)
+    (effects (font (size 1.27 1.27) bold italic) (justify left bottom))
+  )
+  (text "From STM32 \n3.3 High 0v low\n" (at 22.225 86.995 0)
+    (effects (font (size 1.27 1.27) bold italic) (justify left bottom))
+  )
   (hierarchical_label "PUMP_12V" (shape input) (at 132.08 62.23 180)
     (effects (font (size 1.27 1.27)) (justify right))
@@
   (hierarchical_label "PUMP_12V" (shape input) (at 113.03 66.04 180)
     (effects (font (size 1.27 1.27)) (justify right))
+  )
+  (hierarchical_label "Brake_out" (shape input) (at 204.47 82.55 180)
+    (effects (font (size 1.27 1.27) bold italic) (justify right))
   )
   (hierarchical_label "PUMP_CTRL" (shape input) (at 100.965 89.535 270)
@@
   (hierarchical_label "BRAKE_12V" (shape input) (at 189.23 62.23 180)
     (effects (font (size 1.27 1.27)) (justify right))
+  )
+  (symbol (lib_id "power:GND") (at 220.345 82.55 0) (unit 1)
+    (in_bom yes) (on_board yes) (fields_autoplaced)
+    (property "Reference" "#PWR?" (id 0) (at 220.345 88.9 0)
+      (effects (font (size 1.27 1.27)) hide)
+    )
+    (property "Value" "GND" (id 1) (at 220.345 87.63 0))
+    (property "Footprint" "" (id 2) (at 220.345 82.55 0)
+      (effects (font (size 1.27 1.27)) hide)
+    )
+    (property "Datasheet" "" (id 3) (at 220.345 82.55 0)
+      (effects (font (size 1.27 1.27)) hide)
+    )
+    (pin "1")
   )
   (symbol (lib_id "Device:R") (at 43.18 73.66 90) (unit 1)
@@
     (pin "1")
   )
+  (symbol (lib_id "Device:R") (at 210.185 82.55 270) (unit 1)
+    (in_bom yes) (on_board yes)
+    (property "Reference" "R?" (id 0) (at 210.185 76.2 90))
+    (property "Value" "10k" (id 1) (at 210.185 82.55 90))
+    (property "Footprint" "" (id 2) (at 210.185 80.772 90)
+      (effects (font (size 1.27 1.27)) hide)
+    )
+    (property "Datasheet" "~" (id 3) (at 210.185 82.55 0)
+      (effects (font (size 1.27 1.27)) hide)
+    )
+    (pin "1")
+    (pin "2")
+  )
   (symbol (lib_name "BV1HAL45EFJ_1") (lib_id "AERO_Symbols:BV1HAL45EFJ") (at 115.57 70.485 0) (unit 1)
