File: RCB/rear-control-board/FuseBank.kicad_sch (KiCad schematic)
At the start: 10 parts

Commit message: Addded comments
Other:
- note added: "Position of fuses from right(top) to left(bottom)"
Changed lines of the file:
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@@
   (junction (at 74.93 73.025) (diameter 0) (color 0 0 0 0)
+  )
+  (bus_entry (at 172.72 43.18) (size 2.54 2.54)
+    (stroke (width 0) (type default) (color 0 0 0 0))
+  )
+  (bus_entry (at 172.72 50.165) (size 2.54 2.54)
+    (stroke (width 0) (type default) (color 0 0 0 0))
+  )
+  (bus_entry (at 172.72 57.785) (size 2.54 2.54)
+    (stroke (width 0) (type default) (color 0 0 0 0))
+  )
+  (bus_entry (at 172.72 64.135) (size 2.54 2.54)
+    (stroke (width 0) (type default) (color 0 0 0 0))
+  )
+  (bus_entry (at 172.72 71.12) (size 2.54 2.54)
+    (stroke (width 0) (type default) (color 0 0 0 0))
+  )
+  (bus_entry (at 172.72 77.47) (size 2.54 2.54)
+    (stroke (width 0) (type default) (color 0 0 0 0))
+  )
+  (bus_entry (at 172.72 83.185) (size 2.54 2.54)
+    (stroke (width 0) (type default) (color 0 0 0 0))
+  )
+  (bus_entry (at 172.72 90.805) (size 2.54 2.54)
+    (stroke (width 0) (type default) (color 0 0 0 0))
+  )
+  (bus_entry (at 172.72 97.155) (size 2.54 2.54)
+    (stroke (width 0) (type default) (color 0 0 0 0))
   )
   (wire (pts (xy 74.93 73.025) (xy 74.93 79.375))
@@
   )
   (wire (pts (xy 74.93 92.075) (xy 74.93 98.425))
+    (stroke (width 0) (type default) (color 0 0 0 0))
+  )
+  (bus (pts (xy 172.72 71.12) (xy 172.72 77.47))
+    (stroke (width 0) (type default) (color 0 0 0 0))
+  )
+  (bus (pts (xy 172.72 57.785) (xy 172.72 64.135))
     (stroke (width 0) (type default) (color 0 0 0 0))
   )
@@
     (stroke (width 0) (type default) (color 0 0 0 0))
   )
+  (bus (pts (xy 172.72 43.18) (xy 172.72 50.165))
+    (stroke (width 0) (type default) (color 0 0 0 0))
+  )
+  (bus (pts (xy 172.72 50.165) (xy 172.72 57.785))
+    (stroke (width 0) (type default) (color 0 0 0 0))
+  )
+  (bus (pts (xy 172.72 97.155) (xy 172.72 106.68))
+    (stroke (width 0) (type default) (color 0 0 0 0))
+  )
+  (bus (pts (xy 172.72 64.135) (xy 172.72 71.12))
+    (stroke (width 0) (type default) (color 0 0 0 0))
+  )
+  (bus (pts (xy 172.72 83.185) (xy 172.72 90.805))
+    (stroke (width 0) (type default) (color 0 0 0 0))
+  )
   (wire (pts (xy 101.6 92.075) (xy 87.63 92.075))
     (stroke (width 0) (type default) (color 0 0 0 0))
@@
   )
   (wire (pts (xy 101.6 66.675) (xy 87.63 66.675))
+    (stroke (width 0) (type default) (color 0 0 0 0))
+  )
+  (bus (pts (xy 172.72 77.47) (xy 172.72 83.185))
+    (stroke (width 0) (type default) (color 0 0 0 0))
+  )
+  (bus (pts (xy 172.72 90.805) (xy 172.72 97.155))
     (stroke (width 0) (type default) (color 0 0 0 0))
   )
@@
     (effects (font (size 1.27 1.27)) (justify left bottom))
   )
+  (text "Position of fuses from right(top) to left(bottom)" (at 200.025 72.39 0)
+    (effects (font (size 1.27 1.27) bold italic) (justify left bottom))
+  )
   (text "INT_12V goes to the onboard \n5v and 3.3v regulator"
     (at 105.41 57.15 0)
     (effects (font (size 1.27 1.27)) (justify left bottom))
   )
+  (label "Front" (at 175.26 66.675 0)
+    (effects (font (size 1.27 1.27) bold italic) (justify left bottom))
+  )
+  (label "INT_12" (at 175.26 45.72 0)
+    (effects (font (size 1.27 1.27) bold italic) (justify left bottom))
+  )
+  (label "Pump ->BV1HAL" (at 175.26 85.725 0)
+    (effects (font (size 1.27 1.27) bold italic) (justify left bottom))
+  )
+  (label "BRB Loop" (at 175.26 52.705 0)
+    (effects (font (size 1.27 1.27) bold italic) (justify left bottom))
+  )
+  (label "Rear" (at 175.26 60.325 0)
+    (effects (font (size 1.27 1.27) bold italic) (justify left bottom))
+  )
+  (label "Brake -> BV1HAL" (at 175.26 73.66 0)
+    (effects (font (size 1.27 1.27) bold italic) (justify left bottom))
+  )
+  (label "BRB" (at 175.26 93.345 0)
+    (effects (font (size 1.27 1.27) bold italic) (justify left bottom))
+  )
+  (label "Rinehart" (at 175.26 99.695 0)
+    (effects (font (size 1.27 1.27) bold italic) (justify left bottom))
+  )
+  (label "Fan -> BV1Hal" (at 175.26 80.01 0)
+    (effects (font (size 1.27 1.27) bold italic) (justify left bottom))
+  )
   (global_label "INT_12V" (shape output) (at 100.965 60.325 0) (fields_autoplaced)
