File: DCB/interface-board/interface-board.kicad_pcb (KiCad board)
At the start: 2 copper layers, 96.5 x 76.2 mm, 13 parts, among them J1 Conn_01x14, J2 Conn_01x05, SW1 SW_SPST, SW2 SW_SPST, SW3 SW_Push_LED, SW4 SW_Push

Commit message: 5mm Led changed
Parts:
- D1, D2: footprint LED_SMD:LED_0603_1608Metric_Pad1.05x0.95mm_HandSolder -> LED_THT:LED_D5.0mm
Other:
- board text added: "C.Grund 22.031 Dash Interface"
- board text removed: "Colin Grund 1.31"
Changed lines of the file:
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@@
     (pad "" np_thru_hole circle (at 0 0) (size 3.2 3.2) (drill 3.2) (layers *.Cu *.Mask))
   )
-  (footprint "LED_SMD:LED_0603_1608Metric_Pad1.05x0.95mm_HandSolder" (layer "B.Cu")
+  (footprint "LED_THT:LED_D5.0mm" (layer "B.Cu")
     (at 101.6 73.66)
-    (descr "LED SMD 0603 (1608 Metric), square (rectangular) end terminal, IPC_7351 nominal, (Body size source: http://www.tortai-tech.com/upload/download/2011102023233369053.pdf), generated with kicad-footprint-generator")
-    (tags "LED handsolder")
+    (descr "LED, diameter 5.0mm, 2 pins, http://cdn-reichelt.de/documents/datenblatt/A500/LL-504BC2E-009.pdf")
+    (tags "LED diameter 5.0mm 2 pins")
     (property "Sheetfile" "interface-board.kicad_sch")
     (property "Sheetname" "")
-    (attr smd)
-    (fp_text reference "D1" (at 0 -1.27) (layer "B.SilkS")
+    (attr through_hole)
+    (fp_text reference "D1" (at 1.27 3.96 180) (layer "B.SilkS")
       (effects (font (size 1 1) (thickness 0.15)) (justify mirror))
     )
-    (fp_text value "LED" (at 0.508 1.524) (layer "B.Fab")
+    (fp_text value "LED" (at 1.27 -3.96 180) (layer "B.Fab")
       (effects (font (size 1 1) (thickness 0.15)) (justify mirror))
     )
-    (fp_text user "${REFERENCE}" (at 0 0) (layer "B.Fab")
-      (effects (font (size 0.4 0.4) (thickness 0.06)) (justify mirror))
+    (fp_text user "${REFERENCE}" (at 1.25 0 180) (layer "B.Fab")
+      (effects (font (size 0.8 0.8) (thickness 0.2)) (justify mirror))
     )
-    (fp_line (start -1.66 -0.735) (end 0.8 -0.735) (layer "B.SilkS") (width 0.12))
-    (fp_line (start -1.66 0.735) (end -1.66 -0.735) (layer "B.SilkS") (width 0.12))
-    (fp_line (start 0.8 0.735) (end -1.66 0.735) (layer "B.SilkS") (width 0.12))
-    (fp_line (start 1.65 -0.73) (end -1.65 -0.73) (layer "B.CrtYd") (width 0.05))
-    (fp_line (start -1.65 -0.73) (end -1.65 0.73) (layer "B.CrtYd") (width 0.05))
-    (fp_line (start 1.65 0.73) (end 1.65 -0.73) (layer "B.CrtYd") (width 0.05))
-    (fp_line (start -1.65 0.73) (end 1.65 0.73) (layer "B.CrtYd") (width 0.05))
-    (fp_line (start -0.8 0.1) (end -0.8 -0.4) (layer "B.Fab") (width 0.1))
-    (fp_line (start -0.8 -0.4) (end 0.8 -0.4) (layer "B.Fab") (width 0.1))
-    (fp_line (start -0.5 0.4) (end -0.8 0.1) (layer "B.Fab") (width 0.1))
-    (fp_line (start 0.8 -0.4) (end 0.8 0.4) (layer "B.Fab") (width 0.1))
-    (fp_line (start 0.8 0.4) (end -0.5 0.4) (layer "B.Fab") (width 0.1))
-    (pad "1" smd roundrect (at -0.875 0) (size 1.05 0.95) (layers "B.Cu" "B.Paste" "B.Mask") (roundrect_rratio 0.25)
+    (fp_line (start -1.29 1.545) (end -1.29 -1.545) (layer "B.SilkS") (width 0.12))
+    (fp_arc (start -1.29 -1.54483) (mid 2.072002 -2.880433) (end 4.26 0.000462) (layer "B.SilkS") (width 0.12))
+    (fp_arc (start 4.26 -0.000462) (mid 2.072002 2.880433) (end -1.29 1.54483) (layer "B.SilkS") (width 0.12))
+    (fp_circle (center 1.27 0) (end 3.77 0) (layer "B.SilkS") (width 0.12) (fill none))
+    (fp_line (start 4.5 3.25) (end -1.95 3.25) (layer "B.CrtYd") (width 0.05))
+    (fp_line (start -1.95 -3.25) (end 4.5 -3.25) (layer "B.CrtYd") (width 0.05))
+    (fp_line (start -1.95 3.25) (end -1.95 -3.25) (layer "B.CrtYd") (width 0.05))
+    (fp_line (start 4.5 -3.25) (end 4.5 3.25) (layer "B.CrtYd") (width 0.05))
+    (fp_line (start -1.23 1.469694) (end -1.23 -1.469694) (layer "B.Fab") (width 0.1))
+    (fp_arc (start -1.230016 -1.469666) (mid 4.17 -0.000016) (end -1.23 1.469694) (layer "B.Fab") (width 0.1))
+    (fp_circle (center 1.27 0) (end 3.77 0) (layer "B.Fab") (width 0.1) (fill none))
+    (pad "1" thru_hole rect (at 0 0) (size 1.8 1.8) (drill 0.9) (layers *.Cu *.Mask)
       (net 1 "/IMD_LED") (pinfunction "K") (pintype "passive"))
-    (pad "2" smd roundrect (at 0.875 0) (size 1.05 0.95) (layers "B.Cu" "B.Paste" "B.Mask") (roundrect_rratio 0.25)
+    (pad "2" thru_hole circle (at 2.54 0) (size 1.8 1.8) (drill 0.9) (layers *.Cu *.Mask)
       (net 2 "GND") (pinfunction "A") (pintype "passive"))
-    (model "${KICAD6_3DMODEL_DIR}/LED_SMD.3dshapes/LED_0603_1608Metric.wrl"
+    (model "${KICAD6_3DMODEL_DIR}/LED_THT.3dshapes/LED_D5.0mm.wrl"
       (offset (xyz 0 0 0))
       (scale (xyz 1 1 1))
@@
     )
   )
-  (footprint "LED_SMD:LED_0603_1608Metric_Pad1.05x0.95mm_HandSolder" (layer "B.Cu")
+  (footprint "LED_THT:LED_D5.0mm" (layer "B.Cu")
     (at 120.35 73.66)
-    (descr "LED SMD 0603 (1608 Metric), square (rectangular) end terminal, IPC_7351 nominal, (Body size source: http://www.tortai-tech.com/upload/download/2011102023233369053.pdf), generated with kicad-footprint-generator")
-    (tags "LED handsolder")
+    (descr "LED, diameter 5.0mm, 2 pins, http://cdn-reichelt.de/documents/datenblatt/A500/LL-504BC2E-009.pdf")
+    (tags "LED diameter 5.0mm 2 pins")
     (property "Sheetfile" "interface-board.kicad_sch")
     (property "Sheetname" "")
-    (attr smd)
-    (fp_text reference "D2" (at 0 -1.27) (layer "B.SilkS")
+    (attr through_hole)
+    (fp_text reference "D2" (at 1.27 3.96 180) (layer "B.SilkS")
       (effects (font (size 1 1) (thickness 0.15)) (justify mirror))
     )
-    (fp_text value "LED" (at 0.15 1.778) (layer "B.Fab")
+    (fp_text value "LED" (at 1.27 -3.96 180) (layer "B.Fab")
       (effects (font (size 1 1) (thickness 0.15)) (justify mirror))
     )
-    (fp_text user "${REFERENCE}" (at 0 0) (layer "B.Fab")
-      (effects (font (size 0.4 0.4) (thickness 0.06)) (justify mirror))
+    (fp_text user "${REFERENCE}" (at 1.25 0 180) (layer "B.Fab")
+      (effects (font (size 0.8 0.8) (thickness 0.2)) (justify mirror))
     )
-    (fp_line (start 0.8 0.735) (end -1.66 0.735) (layer "B.SilkS") (width 0.12))
-    (fp_line (start -1.66 -0.735) (end 0.8 -0.735) (layer "B.SilkS") (width 0.12))
-    (fp_line (start -1.66 0.735) (end -1.66 -0.735) (layer "B.SilkS") (width 0.12))
-    (fp_line (start -1.65 -0.73) (end -1.65 0.73) (layer "B.CrtYd") (width 0.05))
-    (fp_line (start 1.65 0.73) (end 1.65 -0.73) (layer "B.CrtYd") (width 0.05))
-    (fp_line (start -1.65 0.73) (end 1.65 0.73) (layer "B.CrtYd") (width 0.05))
-    (fp_line (start 1.65 -0.73) (end -1.65 -0.73) (layer "B.CrtYd") (width 0.05))
-    (fp_line (start -0.8 -0.4) (end 0.8 -0.4) (layer "B.Fab") (width 0.1))
-    (fp_line (start -0.8 0.1) (end -0.8 -0.4) (layer "B.Fab") (width 0.1))
-    (fp_line (start 0.8 0.4) (end -0.5 0.4) (layer "B.Fab") (width 0.1))
-    (fp_line (start 0.8 -0.4) (end 0.8 0.4) (layer "B.Fab") (width 0.1))
-    (fp_line (start -0.5 0.4) (end -0.8 0.1) (layer "B.Fab") (width 0.1))
-    (pad "1" smd roundrect (at -0.875 0) (size 1.05 0.95) (layers "B.Cu" "B.Paste" "B.Mask") (roundrect_rratio 0.25)
+    (fp_line (start -1.29 1.545) (end -1.29 -1.545) (layer "B.SilkS") (width 0.12))
+    (fp_arc (start -1.29 -1.54483) (mid 2.072002 -2.880433) (end 4.26 0.000462) (layer "B.SilkS") (width 0.12))
+    (fp_arc (start 4.26 -0.000462) (mid 2.072002 2.880433) (end -1.29 1.54483) (layer "B.SilkS") (width 0.12))
+    (fp_circle (center 1.27 0) (end 3.77 0) (layer "B.SilkS") (width 0.12) (fill none))
+    (fp_line (start -1.95 -3.25) (end 4.5 -3.25) (layer "B.CrtYd") (width 0.05))
+    (fp_line (start 4.5 3.25) (end -1.95 3.25) (layer "B.CrtYd") (width 0.05))
+    (fp_line (start -1.95 3.25) (end -1.95 -3.25) (layer "B.CrtYd") (width 0.05))
+    (fp_line (start 4.5 -3.25) (end 4.5 3.25) (layer "B.CrtYd") (width 0.05))
+    (fp_line (start -1.23 1.469694) (end -1.23 -1.469694) (layer "B.Fab") (width 0.1))
+    (fp_arc (start -1.230016 -1.469666) (mid 4.17 -0.000016) (end -1.23 1.469694) (layer "B.Fab") (width 0.1))
+    (fp_circle (center 1.27 0) (end 3.77 0) (layer "B.Fab") (width 0.1) (fill none))
+    (pad "1" thru_hole rect (at 0 0) (size 1.8 1.8) (drill 0.9) (layers *.Cu *.Mask)
       (net 3 "/AMS_LED") (pinfunction "K") (pintype "passive"))
-    (pad "2" smd roundrect (at 0.875 0) (size 1.05 0.95) (layers "B.Cu" "B.Paste" "B.Mask") (roundrect_rratio 0.25)
+    (pad "2" thru_hole circle (at 2.54 0) (size 1.8 1.8) (drill 0.9) (layers *.Cu *.Mask)
       (net 2 "GND") (pinfunction "A") (pintype "passive"))
-    (model "${KICAD6_3DMODEL_DIR}/LED_SMD.3dshapes/LED_0603_1608Metric.wrl"
+    (model "${KICAD6_3DMODEL_DIR}/LED_THT.3dshapes/LED_D5.0mm.wrl"
       (offset (xyz 0 0 0))
       (scale (xyz 1 1 1))
@@
       (xy 127 66.04)
     ) (layer "Edge.Cuts") (width 0.1) (fill none))
-  (gr_text "Colin Grund\n1.31" (at 111.252 72.136) (layer "B.Cu")
+  (gr_text "C.Grund\n22.031\nDash Interface\n" (at 111.252 72.136) (layer "F.SilkS")
     (effects (font (size 1.5 1.5) (thickness 0.3)))
   )
