File: DCB/interface-board/interface-board.kicad_sch (KiCad schematic)
At the start: 12 parts, among them J1 Conn_01x14, J2 Conn_01x05, SW1 SW_SPST, SW2 SW_SPST, SW3 SW_Push_LED, SW4 SW_Push

Commit message: 5mm Led changed
Parts:
- D1, D2: footprint LED_SMD:LED_0603_1608Metric_Pad1.05x0.95mm_HandSolder -> LED_THT:LED_D5.0mm
Changed lines of the file:
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@@
       (effects (font (size 1.27 1.27)) (justify left))
     )
-    (property "Footprint" "LED_SMD:LED_0603_1608Metric_Pad1.05x0.95mm_HandSolder" (id 2) (at 118.11 60.96 0)
+    (property "Footprint" "LED_THT:LED_D5.0mm" (id 2) (at 118.11 60.96 0)
       (effects (font (size 1.27 1.27)) hide)
     )
@@
       (effects (font (size 1.27 1.27)) (justify left))
     )
-    (property "Footprint" "LED_SMD:LED_0603_1608Metric_Pad1.05x0.95mm_HandSolder" (id 2) (at 137.16 60.96 0)
+    (property "Footprint" "LED_THT:LED_D5.0mm" (id 2) (at 137.16 60.96 0)
       (effects (font (size 1.27 1.27)) hide)
     )
@@
     )
     (path "/00000000-0000-0000-0000-000062083cc8"
-      (reference "D1") (unit 1) (value "LED") (footprint "LED_SMD:LED_0603_1608Metric_Pad1.05x0.95mm_HandSolder")
+      (reference "D1") (unit 1) (value "LED") (footprint "LED_THT:LED_D5.0mm")
     )
     (path "/00000000-0000-0000-0000-0000620840b4"
-      (reference "D2") (unit 1) (value "LED") (footprint "LED_SMD:LED_0603_1608Metric_Pad1.05x0.95mm_HandSolder")
+      (reference "D2") (unit 1) (value "LED") (footprint "LED_THT:LED_D5.0mm")
     )
     (path "/f1084b0d-b992-4d4c-9074-1c148a908ad5"
