File: DCB/interface-board/interface-board.kicad_sch (KiCad schematic)
At the start: 12 parts, among them J1 Conn_01x14, J2 Conn_01x05, SW1 SW_SPST, SW2 SW_SPST, SW3 SW_Push_LED, SW4 SW_Push

Commit message: Surface mount dash
Parts:
- removed H1, H2: MountingHole, MountingHole:MountingHole_3.2mm_M3, symbol Mechanical:MountingHole
- removed J1: Conn_01x14, AERO_Footprints:TE_1-776262-1_14pin_Vertical, symbol Connector_Generic:Conn_01x14
- removed J2: Conn_01x05, Connector_JST:JST_XH_S5B-XH-A-1_1x05_P2.50mm_Horizontal, symbol Connector_Generic:Conn_01x05
- added J1: Conn_01x05, Connector_JST:JST_XH_S5B-XH-A_1x05_P2.50mm_Horizontal, symbol Connector_Generic:Conn_01x05
- added J2: Conn_01x04, Connector_JST:JST_XH_S4B-XH-A_1x04_P2.50mm_Horizontal, symbol Connector_Generic:Conn_01x04
- added J3: Conn_01x02, Connector_JST:JST_XH_S2B-XH-A_1x02_P2.50mm_Horizontal, symbol Connector_Generic:Conn_01x02
- RV1, RV2: footprint Connector_JST:JST_XH_S3B-XH-A-1_1x03_P2.50mm_Horizontal -> AERO_Footprints:SMD_Pot
- SW3: footprint Connector_JST:JST_XH_S4B-XH-A-1_1x04_P2.50mm_Horizontal -> AERO_Footprints:LED_PUSHBUTTON
- SW4: footprint Connector_JST:JST_XH_S2B-XH-A-1_1x02_P2.50mm_Horizontal -> Button_Switch_THT:SW_PUSH_6mm
Connections:
- net +5V: now also J1.3 (Pin_3)
- net AMS_LED: now also J1.2 (Pin_2)
- net GND: now also J1.1 (Pin_1)
- net IMD_LED: now also J2.4 (Pin_4)
- net LCD_BTN: now also J2.1 (Pin_1)
- net POT_BRAKE: now also J1.4 (Pin_4)
- net POT_REGEN: now also J1.5 (Pin_5)
- net RTD_LED: now also J3.2 (Pin_2)
- net START_BTN: now also J3.1 (Pin_1)
- net SW_COOLING: now also J2.3 (Pin_3)
- net SW_DIRECTION: now also J2.2 (Pin_2)
Other:
- note removed: "Driver Interface"
- note removed: "To LCD Panel"
