File: DCB/interface-board/interface-board.kicad_sch (KiCad schematic)
At the start: 12 parts, among them J1 Conn_01x14, J2 Conn_01x05, SW1 SW_SPST, SW2 SW_SPST, SW3 SW_Push_LED, SW4 SW_Push

Commit message: Addded comments
Parts:
- added D?: D, symbol Device:D
- added R?: 330, symbol Device:R
Connections:
- net GND: now also D?.1 (K)
- new net: D?.2 (A), R?.2
- new net IMD_IND: R?.1
Other:
- note added: "3.3v from DCB need 5 for LCD"
- note added: "Addition"
- note added: "Backwards. 3.3v is coming from microcontroler"
Changed lines of the file:
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@@
+    (stroke (width 0) (type default) (color 0 0 0 0))
+  )
+  (polyline (pts (xy 52.07 73.66) (xy 52.07 46.355))
     (stroke (width 0) (type default) (color 0 0 0 0))
   )
@@
     (stroke (width 0) (type default) (color 0 0 0 0))
   )
+  (polyline (pts (xy 84.455 46.355) (xy 84.455 73.66))
+    (stroke (width 0) (type default) (color 0 0 0 0))
+  )
+  (wire (pts (xy 74.295 57.785) (xy 74.295 59.055))
+    (stroke (width 0) (type default) (color 0 0 0 0))
+  )
   (wire (pts (xy 160.02 71.12) (xy 160.02 64.77))
     (stroke (width 0) (type default) (color 0 0 0 0))
@@
     (stroke (width 0) (type default) (color 0 0 0 0))
   )
+  (wire (pts (xy 67.31 51.435) (xy 74.295 51.435))
+    (stroke (width 0) (type default) (color 0 0 0 0))
+  )
   (wire (pts (xy 157.48 52.07) (xy 144.78 52.07))
     (stroke (width 0) (type default) (color 0 0 0 0))
   )
+  (polyline (pts (xy 52.07 46.355) (xy 84.455 46.355))
+    (stroke (width 0) (type default) (color 0 0 0 0))
+  )
   (wire (pts (xy 52.07 91.44) (xy 66.04 91.44))
     (stroke (width 0) (type default) (color 0 0 0 0))
@@
     (stroke (width 0) (type default) (color 0 0 0 0))
   )
+  (polyline (pts (xy 84.455 73.66) (xy 52.07 73.66))
+    (stroke (width 0) (type default) (color 0 0 0 0))
+  )
   (wire (pts (xy 238.76 62.23) (xy 251.46 62.23))
     (stroke (width 0) (type default) (color 0 0 0 0))
@@
     (stroke (width 0) (type default) (color 0 0 0 0))
   )
+  (text "3.3v from DCB\nneed 5 for LCD" (at 215.9 34.925 0)
+    (effects (font (size 1.27 1.27) bold italic) (justify left bottom))
+  )
+  (text "Addition" (at 63.5 45.72 0)
+    (effects (font (size 1.27 1.27) (thickness 0.254) bold italic) (justify left bottom))
+  )
   (text "To LCD Panel " (at 242.57 85.09 0)
     (effects (font (size 1.27 1.27)) (justify left bottom))
   )
+  (text "Backwards. 3.3v is coming from microcontroler " (at 115.57 45.72 0)
+    (effects (font (size 1.27 1.27) (thickness 0.254) bold italic) (justify left bottom))
+  )
   (text "Driver Interface" (at 246.38 31.75 0)
     (effects (font (size 1.27 1.27)) (justify left bottom))
@@
   (label "RTD_LED" (at 238.76 41.91 0)
     (effects (font (size 1.27 1.27)) (justify left bottom))
+  )
+  (label "IMD_IND" (at 67.31 51.435 180)
+    (effects (font (size 1.27 1.27)) (justify right bottom))
   )
   (label "START_BTN" (at 173.99 52.07 180)
@@
     (pin "1")
   )
+  (symbol (lib_id "power:GND") (at 74.295 65.405 0) (unit 1)
+    (in_bom yes) (on_board yes) (fields_autoplaced)
+    (property "Reference" "#PWR?" (id 0) (at 74.295 71.755 0)
+      (effects (font (size 1.27 1.27)) hide)
+    )
+    (property "Value" "GND" (id 1) (at 74.295 69.85 0))
+    (property "Footprint" "" (id 2) (at 74.295 65.405 0)
+      (effects (font (size 1.27 1.27)) hide)
+    )
+    (property "Datasheet" "" (id 3) (at 74.295 65.405 0)
+      (effects (font (size 1.27 1.27)) hide)
+    )
+    (pin "1")
+  )
   (symbol (lib_id "Mechanical:MountingHole") (at 30.48 174.625 0) (unit 1)
     (in_bom yes) (on_board yes)
@@
       (effects (font (size 1.27 1.27)) hide)
     )
+  )
+  (symbol (lib_id "Device:D") (at 74.295 61.595 90) (unit 1)
+    (in_bom yes) (on_board yes) (fields_autoplaced)
+    (property "Reference" "D?" (id 0) (at 77.47 60.3249 90)
+      (effects (font (size 1.27 1.27)) (justify right))
+    )
+    (property "Value" "D" (id 1) (at 77.47 62.8649 90)
+      (effects (font (size 1.27 1.27)) (justify right))
+    )
+    (property "Footprint" "" (id 2) (at 74.295 61.595 0)
+      (effects (font (size 1.27 1.27)) hide)
+    )
+    (property "Datasheet" "~" (id 3) (at 74.295 61.595 0)
+      (effects (font (size 1.27 1.27)) hide)
+    )
+    (pin "1")
+    (pin "2")
+  )
+  (symbol (lib_id "Device:R") (at 74.295 55.245 0) (unit 1)
+    (in_bom yes) (on_board yes)
+    (property "Reference" "R?" (id 0) (at 76.2 53.9749 0)
+      (effects (font (size 1.27 1.27)) (justify left))
+    )
+    (property "Value" "330" (id 1) (at 74.295 57.15 90)
+      (effects (font (size 1.27 1.27)) (justify left))
+    )
+    (property "Footprint" "" (id 2) (at 72.517 55.245 90)
+      (effects (font (size 1.27 1.27)) hide)
+    )
+    (property "Datasheet" "~" (id 3) (at 74.295 55.245 0)
+      (effects (font (size 1.27 1.27)) hide)
+    )
+    (pin "1")
+    (pin "2")
   )
   (symbol (lib_id "Mechanical:MountingHole") (at 30.48 165.1 0) (unit 1)
@@
       (reference "#PWR0109") (unit 1) (value "GND") (footprint "")
     )
+    (path "/31bf73f8-5ead-4618-bd11-6325766f2985"
+      (reference "#PWR?") (unit 1) (value "GND") (footprint "")
+    )
     (path "/00000000-0000-0000-0000-000062083cc8"
       (reference "D1") (unit 1) (value "LED") (footprint "LED_SMD:LED_0603_1608Metric_Pad1.05x0.95mm_HandSolder")
@@
       (reference "D2") (unit 1) (value "LED") (footprint "LED_SMD:LED_0603_1608Metric_Pad1.05x0.95mm_HandSolder")
     )
+    (path "/684829a1-14fb-436a-9093-a9211cbef360"
+      (reference "D?") (unit 1) (value "D") (footprint "")
+    )
     (path "/f1084b0d-b992-4d4c-9074-1c148a908ad5"
       (reference "H1") (unit 1) (value "MountingHole") (footprint "MountingHole:MountingHole_3.2mm_M3")
@@
       (reference "J2") (unit 1) (value "Conn_01x05") (footprint "Connector_JST:JST_XH_S5B-XH-A-1_1x05_P2.50mm_Horizontal")
     )
+    (path "/8f40cd30-616e-41e2-bee9-266c3138b0af"
+      (reference "R?") (unit 1) (value "330") (footprint "")
+    )
     (path "/00000000-0000-0000-0000-000062084c31"
