File: DCB/driver-control-board/driver-control-board.kicad_pcb (KiCad board)
At the start: 2 copper layers, 95.5 x 61 mm, 34 parts, among them J2 Conn_01x14, J3 Conn_01x08, J4 Conn_01x23, J5 Conn_02x10_Counter_Clockwise, J6 Conn_01x14, J7 FTSH-107-01-F-DV-K, Q1 2N7002, U1 STM32F413CGUx, U3 LDL1117S33R, U4 MAX33054EASA+T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

Commit message: finished schem and layout. Ready for Review
Parts:
- added G***: LOGO, AERO_Footprints:AERO_Logo_10x4mm, F.Cu at (106.2, 96.5)
- moved D1 8.29 mm to (114.8, 112.3), turned to 0 degrees
- moved U3 4.91 mm to (115.6, 105.9), turned to 180 degrees
- moved C6 4.54 mm to (120.9, 108.5), turned to -90 degrees
- moved R2 3.90 mm to (114.8, 110.5), turned to 180 degrees
- moved C1 3.40 mm to (120.9, 104.9), turned to -90 degrees
Connections:
- J2 pad 14: +5V -> +3V3
- J4 pad 16: +3V3 -> +12V
- J4 pad 19: +12V -> +3V3
Routing:
- net +3V3: track 15.5 -> 249.5 mm, vias 3 -> 11
- net +12V: track 37.9 -> 96.3 mm
- net Net-(D1-Pad2): track 0.00 -> 1.79 mm
- net /IMD_LED: track 27.1 -> 25.8 mm
- net GND: track 23.7 -> 22.6 mm, vias 14 -> 29
- net /SW_DIRECTION: track 24.9 -> 23.9 mm
Other:
- board text added: "DCB"
- board text added: "G.Spearing 20.044"
