File: DCB/driver-control-board/driver-control-board.kicad_sch (KiCad schematic)
At the start: 34 parts, among them J2 Conn_01x14, J3 Conn_01x08, J4 Conn_01x23, J5 Conn_02x10_Counter_Clockwise, J6 Conn_01x14, J7 FTSH-107-01-F-DV-K, Q1 2N7002, U1 STM32F413CGUx, U3 LDL1117S33R, U4 MAX33054EASA+T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

Commit message: touching up layout and making gerbers
Connections:
- net +3V3: now also J4.19 (Pin_19)
- net GND: now also J4.1 (Pin_1)
Changed lines of the file:
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@@
   (junction (at 242.57 61.595) (diameter 0) (color 0 0 0 0)
+  )
+  (junction (at 242.57 64.135) (diameter 0) (color 0 0 0 0)
   )
   (junction (at 245.745 103.505) (diameter 0) (color 0 0 0 0)
@@
     (stroke (width 0) (type default) (color 0 0 0 0))
   )
+  (wire (pts (xy 242.57 66.675) (xy 242.57 64.135))
+    (stroke (width 0) (type default) (color 0 0 0 0))
+  )
   (wire (pts (xy 207.645 62.23) (xy 220.345 62.23))
     (stroke (width 0) (type default) (color 0 0 0 0))
@@
     (stroke (width 0) (type default) (color 0 0 0 0))
   )
+  (wire (pts (xy 241.935 20.955) (xy 241.935 23.495))
+    (stroke (width 0) (type default) (color 0 0 0 0))
+  )

Commit message: Addded comments
Other:
- note added: "Buzzer is soldered to 4 and 16 on J4"
- note added: "Check part footprint RN1 seems wrong?"
- note added: "GND to Frame"
- note added: "Yes Do not ground interface board to frame"
Changed lines of the file:
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@@
     (effects (font (size 1.27 1.27)) (justify left bottom))
+  )
+  (text "Check part footprint \nRN1 seems wrong?" (at 15.24 191.135 0)
+    (effects (font (size 1.27 1.27) (thickness 0.254) bold italic) (justify left bottom))
   )
   (text "RX" (at 167.005 46.355 0)
@@
   (text "Buzzer, Low Side Drive" (at 85.09 22.86 0)
     (effects (font (size 1.27 1.27)) (justify left bottom))
+  )
+  (text "Yes Do not ground\ninterface board to frame " (at 200.66 27.305 0)
+    (effects (font (size 1.27 1.27) bold italic) (justify left bottom))
   )
   (text "Driver Interface" (at 215.265 29.21 0)
@@
     (effects (font (size 1.27 1.27)) (justify left bottom))
   )
+  (text "Buzzer is \nsoldered to \n4 and 16 on J4\n" (at 268.605 31.75 0)
+    (effects (font (size 1.27 1.27) (thickness 0.254) bold italic) (justify left bottom))
+  )
   (text "Power Regulation" (at 60.96 24.13 180)
     (effects (font (size 2.9972 2.9972)) (justify right bottom))
@@
     (effects (font (size 1.27 1.27)) (justify left bottom))
   )
+  (text "GND to Frame" (at 150.495 57.785 0)
+    (effects (font (size 1.27 1.27) bold italic) (justify left bottom))
+  )
   (text "STBY logic low is normal mode\nlogic high is receive only"
