File: PAM/pacman/pacman.kicad_pcb (KiCad board)
At the start: 2 copper layers, 92.7 x 66 mm, 23 parts, among them J1 Conn_01x08, J2 Conn_01x04, J3 Conn_01x01, J4 Conn_01x01, J5 Conn_01x01, J6 Conn_01x02, J9 JST PH, K1 G2RL, K2 G5V-1, K3 G5V-1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

Commit message: touching up layout and making gerbers
Changed lines of the file:
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@@
       (outputformat 1)
       (mirror false)
-      (drillshape 1)
+      (drillshape 0)
       (scaleselection 1)
-      (outputdirectory "")
+      (outputdirectory "Pac1_Gerber/")
     )
   )
@@
     (fp_line (start 7.95 -1.7) (end -1.95 -1.7) (layer "F.Fab") (width 0.1))
     (fp_line (start 7.95 2.8) (end 7.95 -1.7) (layer "F.Fab") (width 0.1))
-    (pad "1" thru_hole roundrect locked (at 0 0 90) (size 1.2 1.75) (drill 0.75) (layers *.Cu *.Mask) (roundrect_rratio 0.208333)
+    (pad "1" thru_hole roundrect locked (at 0 0 90) (size 1.2 1.75) (drill 0.75) (layers *.Cu *.Mask) (roundrect_rratio 0.2083333333)
       (net 12 "/AIR_B-") (pinfunction "Pin_1") (pintype "passive"))
     (pad "2" thru_hole oval locked (at 2 0 90) (size 1.2 1.75) (drill 0.75) (layers *.Cu *.Mask)
@@
     (fp_line (start 0 -1.35) (end 0.625 -2.35) (layer "F.Fab") (width 0.1))
     (fp_line (start 9.95 -2.35) (end -2.45 -2.35) (layer "F.Fab") (width 0.1))
-    (pad "1" thru_hole roundrect locked (at 0 0 90) (size 1.7 1.95) (drill 0.95) (layers *.Cu *.Mask) (roundrect_rratio 0.147059)
+    (pad "1" thru_hole roundrect locked (at 0 0 90) (size 1.7 1.95) (drill 0.95) (layers *.Cu *.Mask) (roundrect_rratio 0.1470588235)
       (net 10 "+12V") (pinfunction "Pin_1") (pintype "passive"))
     (pad "2" thru_hole oval locked (at 2.5 0 90) (size 1.7 1.95) (drill 0.95) (layers *.Cu *.Mask)
@@
     (fp_line (start -3.1 4.05) (end -3.1 -3.95) (layer "F.Fab") (width 0.1))
     (pad "" np_thru_hole circle locked (at -1.5 3.25 90) (size 1.6 1.6) (drill 1.6) (layers *.Cu *.Mask))
-    (pad "1" thru_hole roundrect locked (at 0 0 90) (size 2.46 2.8) (drill 1.8) (layers *.Cu *.Mask) (roundrect_rratio 0.101626)
+    (pad "1" thru_hole roundrect locked (at 0 0 90) (size 2.46 2.8) (drill 1.8) (layers *.Cu *.Mask) (roundrect_rratio 0.1016260163)
       (net 15 "/INT+") (pinfunction "Pin_1") (pintype "passive"))
     (model "${KICAD6_3DMODEL_DIR}/Connector_Hirose.3dshapes/Hirose_DF63M-1P-3.96DSA_1x01_P3.96mm_Vertical.wrl"
@@
     (fp_line (start 4.95 -2.35) (end -2.45 -2.35) (layer "F.Fab") (width 0.1))
     (fp_line (start 0 -1.35) (end 0.625 -2.35) (layer "F.Fab") (width 0.1))
-    (pad "1" thru_hole roundrect locked (at 0 0 270) (size 1.7 2) (drill 1) (layers *.Cu *.Mask) (roundrect_rratio 0.147059)
+    (pad "1" thru_hole roundrect locked (at 0 0 270) (size 1.7 2) (drill 1) (layers *.Cu *.Mask) (roundrect_rratio 0.1470588235)
       (net 19 "Net-(F3-Pad2)") (pinfunction "Pin_1") (pintype "passive"))
     (pad "2" thru_hole oval locked (at 2.5 0 270) (size 1.7 2) (drill 1) (layers *.Cu *.Mask)
@@
     (fp_line (start -3.1 -3.95) (end -1.9 -3.95) (layer "F.Fab") (width 0.1))
     (pad "" np_thru_hole circle locked (at -1.5 3.25) (size 1.6 1.6) (drill 1.6) (layers *.Cu *.Mask))
-    (pad "1" thru_hole roundrect locked (at 0 0) (size 2.46 2.8) (drill 1.8) (layers *.Cu *.Mask) (roundrect_rratio 0.101626)
+    (pad "1" thru_hole roundrect locked (at 0 0) (size 2.46 2.8) (drill 1.8) (layers *.Cu *.Mask) (roundrect_rratio 0.1016260163)
       (net 9 "/B+") (pinfunction "Pin_1") (pintype "passive"))
     (model "${KICAD6_3DMODEL_DIR}/Connector_Hirose.3dshapes/Hirose_DF63M-1P-3.96DSA_1x01_P3.96mm_Vertical.wrl"
@@
     (fp_line (start 3.1 -3.95) (end 1.9 -3.95) (layer "F.Fab") (width 0.1))
     (pad "" np_thru_hole circle locked (at -1.5 3.25 90) (size 1.6 1.6) (drill 1.6) (layers *.Cu *.Mask))
-    (pad "1" thru_hole roundrect locked (at 0 0 90) (size 2.46 2.8) (drill 1.8) (layers *.Cu *.Mask) (roundrect_rratio 0.101626)
+    (pad "1" thru_hole roundrect locked (at 0 0 90) (size 2.46 2.8) (drill 1.8) (layers *.Cu *.Mask) (roundrect_rratio 0.1016260163)
       (net 1 "/INT-") (pinfunction "Pin_1") (pintype "passive"))
     (model "${KICAD6_3DMODEL_DIR}/Connector_Hirose.3dshapes/Hirose_DF63M-1P-3.96DSA_1x01_P3.96mm_Vertical.wrl"
