File: PAM/pacman_side_2/pacman_side_2.kicad_sch (KiCad schematic)
At the start: 23 parts, among them J1 Conn_01x08, J2 Conn_01x04, J3 Conn_01x01, J4 Conn_01x01, J5 Conn_01x01, J6 Conn_01x02, J9 JST PH, K1 G2RL, K2 G5V-1, K3 G5V-1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

Commit message: Adding CAN termination resistors
Parts:
- added R2: 120, Resistor_SMD:R_0603_1608Metric_Pad0.98x0.95mm_HandSolder, symbol Device:R
Connections:
- net BMS_CAN+: now also R2.1
- net BMS_CAN-: now also R2.2
Other:
- note added: "Optional Termination Resistor"
Changed lines of the file:
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@@
+    (stroke (width 0) (type default) (color 0 0 0 0))
+  )
+  (wire (pts (xy 48.895 132.08) (xy 53.975 132.08))
     (stroke (width 0) (type default) (color 0 0 0 0))
   )
@@
     (stroke (width 0) (type default) (color 0 0 0 0))
   )
+  (wire (pts (xy 48.895 137.16) (xy 48.895 139.7))
+    (stroke (width 0) (type default) (color 0 0 0 0))
+  )
   (wire (pts (xy 142.24 59.69) (xy 142.24 57.15))
     (stroke (width 0) (type default) (color 0 0 0 0))
@@
     (stroke (width 0) (type default) (color 0 0 0 0))
   )
-  (wire (pts (xy 35.56 134.62) (xy 46.99 134.62))
-    (stroke (width 0) (type default) (color 0 0 0 0))
-  )
   (polyline (pts (xy 123.19 73.66) (xy 123.19 91.44))
     (stroke (width 0) (type default) (color 0 0 0 0))
@@
     (stroke (width 0) (type default) (color 0 0 0 0))
   )
+  (wire (pts (xy 48.895 134.62) (xy 48.895 132.08))
+    (stroke (width 0) (type default) (color 0 0 0 0))
+  )
   (wire (pts (xy 171.45 82.55) (xy 172.72 82.55))
     (stroke (width 0) (type default) (color 0 0 0 0))
@@
     (stroke (width 0) (type default) (color 0 0 0 0))
   )
-  (wire (pts (xy 35.56 137.16) (xy 46.99 137.16))
+  (wire (pts (xy 35.56 137.16) (xy 48.895 137.16))
     (stroke (width 0) (type default) (color 0 0 0 0))
   )
@@
     (stroke (width 0) (type default) (color 0 0 0 0))
   )
+  (wire (pts (xy 35.56 134.62) (xy 48.895 134.62))
+    (stroke (width 0) (type default) (color 0 0 0 0))
+  )
   (wire (pts (xy 118.745 184.15) (xy 109.855 184.15))
     (stroke (width 0) (type default) (color 0 0 0 0))
@@
   )
   (wire (pts (xy 237.49 85.09) (xy 237.49 92.71))
+    (stroke (width 0) (type default) (color 0 0 0 0))
+  )
+  (wire (pts (xy 48.895 139.7) (xy 53.975 139.7))
     (stroke (width 0) (type default) (color 0 0 0 0))
   )
@@
   (text "Energy dissipated by 2 resistors when charging bus\ncapacitance (ONLY MOTOR CONTROLLER, FOR\nNOW): 20.7 Joules\n\nEnergy dissipated by 1 resistor: 20.7/2 Joules\n\nEquivalent pulse length: 0.25 seconds @ 288 Volts\n\nDatasheet specs 1000 Volt maximum for 0.25\nsecond pulse (so this resistor will work)"
     (at 96.52 125.73 0)
+    (effects (font (size 1.27 1.27)) (justify left bottom))
+  )
+  (text "Optional Termination\nResistor" (at 53.34 130.81 0)
     (effects (font (size 1.27 1.27)) (justify left bottom))
   )
@@
     (pin "9")
   )
+  (symbol (lib_id "Device:R") (at 53.975 135.89 0) (unit 1)
+    (in_bom yes) (on_board yes) (fields_autoplaced)
+    (property "Reference" "R2" (id 0) (at 55.88 134.6199 0)
+      (effects (font (size 1.27 1.27)) (justify left))
+    )
+    (property "Value" "120" (id 1) (at 55.88 137.1599 0)
+      (effects (font (size 1.27 1.27)) (justify left))
+    )
+    (property "Footprint" "Resistor_SMD:R_0603_1608Metric_Pad0.98x0.95mm_HandSolder" (id 2) (at 52.197 135.89 90)
+      (effects (font (size 1.27 1.27)) hide)
+    )
+    (property "Datasheet" "~" (id 3) (at 53.975 135.89 0)
+      (effects (font (size 1.27 1.27)) hide)
+    )
+    (pin "1")
+    (pin "2")
+  )
   (symbol (lib_id "Connector_Generic:Conn_01x01") (at 26.67 35.56 180) (unit 1)
     (in_bom yes) (on_board yes) (fields_autoplaced)
@@
       (reference "R1") (unit 1) (value "39k") (footprint "Resistor_THT:R_Axial_DIN0414_L11.9mm_D4.5mm_P25.40mm_Horizontal")
     )
+    (path "/5f7505cc-53a6-463b-b397-33ff845b1ac0"
+      (reference "R2") (unit 1) (value "120") (footprint "Resistor_SMD:R_0603_1608Metric_Pad0.98x0.95mm_HandSolder")
+    )
     (path "/00000000-0000-0000-0000-00005c5151c5"

Commit message: Major Review and Part Update
updating footprints, component values, layouts
Parts:
- removed R4, R7: 1k 7W, Resistor_THT:R_Axial_Power_L25.0mm_W9.0mm_P30.48mm, symbol Device:R_US
- added R3: 500, Package_TO_SOT_THT:TO-220-2_Horizontal_TabDown, symbol Device:R
Connections:
- net INT+: now also R3.1
- net at K1.5, K1.6: now also R3.2
Other:
- note added: "20W"
Changed lines of the file:
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@@
   (junction (at 227.33 77.47) (diameter 0) (color 0 0 0 0)
   )
-  (junction (at 124.46 83.82) (diameter 0) (color 0 0 0 0)
-  )
   (junction (at 172.72 82.55) (diameter 0) (color 0 0 0 0)
   )
@@
   (junction (at 154.94 76.2) (diameter 0) (color 0 0 0 0)
   )
-  (junction (at 134.62 80.01) (diameter 0) (color 0 0 0 0)
-  )
   (junction (at 237.49 85.09) (diameter 0) (color 0 0 0 0)
   )
@@
     (stroke (width 0) (type default) (color 0 0 0 0))
   )
-  (wire (pts (xy 124.46 83.82) (xy 124.46 80.01))
-    (stroke (width 0) (type default) (color 0 0 0 0))
-  )
   (wire (pts (xy 132.08 57.15) (xy 125.73 57.15))
     (stroke (width 0) (type default) (color 0 0 0 0))
   )
-  (wire (pts (xy 124.46 83.82) (xy 111.76 83.82))
+  (wire (pts (xy 124.46 80.01) (xy 116.84 80.01))
     (stroke (width 0) (type default) (color 0 0 0 0))
   )
@@
     (stroke (width 0) (type default) (color 0 0 0 0))
   )
-  (wire (pts (xy 134.62 87.63) (xy 134.62 80.01))
-    (stroke (width 0) (type default) (color 0 0 0 0))
-  )
   (wire (pts (xy 31.75 35.56) (xy 39.37 35.56))
     (stroke (width 0) (type default) (color 0 0 0 0))
   )
-  (wire (pts (xy 132.08 87.63) (xy 134.62 87.63))
-    (stroke (width 0) (type default) (color 0 0 0 0))
-  )
   (wire (pts (xy 154.94 92.71) (xy 163.83 92.71))
     (stroke (width 0) (type default) (color 0 0 0 0))
@@
     (stroke (width 0) (type default) (color 0 0 0 0))
   )
-  (wire (pts (xy 134.62 80.01) (xy 144.78 80.01))
+  (wire (pts (xy 132.08 80.01) (xy 144.78 80.01))
     (stroke (width 0) (type default) (color 0 0 0 0))
   )
@@
     (stroke (width 0) (type default) (color 0 0 0 0))
   )
-  (wire (pts (xy 124.46 83.82) (xy 124.46 87.63))
-    (stroke (width 0) (type default) (color 0 0 0 0))
-  )
   (wire (pts (xy 184.15 105.41) (xy 184.15 102.87))
     (stroke (width 0) (type default) (color 0 0 0 0))
@@
   )
   (wire (pts (xy 142.24 57.15) (xy 139.7 57.15))
-    (stroke (width 0) (type default) (color 0 0 0 0))
-  )
-  (wire (pts (xy 132.08 80.01) (xy 134.62 80.01))
     (stroke (width 0) (type default) (color 0 0 0 0))
   )
@@
     (effects (font (size 1.27 1.27)) (justify left bottom))
   )
+  (text "20W\n" (at 127 84.455 0)
+    (effects (font (size 1.27 1.27)) (justify left bottom))
+  )
   (text "39k, 3W resistor" (at 41.91 81.28 0)
     (effects (font (size 1.27 1.27)) (justify left bottom))
@@
     (effects (font (size 1.27 1.27)) (justify right bottom))
   )
-  (label "INT+" (at 111.76 83.82 0)
+  (label "INT+" (at 116.84 80.01 0)
     (effects (font (size 1.27 1.27)) (justify left bottom))
   )
@@
     (pin "1")
   )
-  (symbol (lib_id "Device:R_US") (at 128.27 80.01 270) (unit 1)
-    (in_bom yes) (on_board yes)
-    (property "Reference" "R4" (id 0) (at 128.27 74.803 90))
-    (property "Value" "1k 7W" (id 1) (at 128.27 77.1144 90))
-    (property "Footprint" "Resistor_THT:R_Axial_Power_L25.0mm_W9.0mm_P30.48mm" (id 2) (at 128.016 81.026 90)
-      (effects (font (size 1.27 1.27)) hide)
-    )
-    (property "Datasheet" "~" (id 3) (at 128.27 80.01 0)
-      (effects (font (size 1.27 1.27)) hide)
-    )
-    (property "MFR P/N" "AC07000001001JAC00" (id 4) (at 128.27 80.01 90)
-      (effects (font (size 1.27 1.27)) hide)
-    )
-    (pin "1")
-    (pin "2")
-  )
   (symbol (lib_id "Device:Q_NPN_BEC") (at 157.48 82.55 0) (mirror y) (unit 1)
     (in_bom yes) (on_board yes)
@@
     )
     (property "Datasheet" "http://www.nxp.com/documents/data_sheet/1N4148_1N4448.pdf" (id 3) (at 207.01 113.03 0)
-      (effects (font (size 1.27 1.27)) hide)
-    )
-    (pin "1")
-    (pin "2")
-  )
-  (symbol (lib_id "Device:R_US") (at 128.27 87.63 270) (unit 1)
-    (in_bom yes) (on_board yes)
-    (property "Reference" "R7" (id 0) (at 128.27 82.423 90))
-    (property "Value" "1k 7W" (id 1) (at 128.27 84.7344 90))
-    (property "Footprint" "Resistor_THT:R_Axial_Power_L25.0mm_W9.0mm_P30.48mm" (id 2) (at 128.016 88.646 90)
-      (effects (font (size 1.27 1.27)) hide)
-    )
-    (property "Datasheet" "~" (id 3) (at 128.27 87.63 0)
-      (effects (font (size 1.27 1.27)) hide)
-    )
-    (property "MFR P/N" "AC07000001001JAC00" (id 4) (at 128.27 87.63 90)
       (effects (font (size 1.27 1.27)) hide)
     )
@@
     (pin "1")
   )
+  (symbol (lib_id "Device:R") (at 128.27 80.01 90) (unit 1)
+    (in_bom yes) (on_board yes)
+    (property "Reference" "R3" (id 0) (at 128.27 77.47 90))
+    (property "Value" "500" (id 1) (at 128.27 80.01 90))
+    (property "Footprint" "Package_TO_SOT_THT:TO-220-2_Horizontal_TabDown" (id 2) (at 128.27 81.788 90)
+      (effects (font (size 1.27 1.27)) hide)
+    )
+    (property "Datasheet" "~" (id 3) (at 128.27 80.01 0)
+      (effects (font (size 1.27 1.27)) hide)
+    )
+    (pin "1")
+    (pin "2")
+  )
   (symbol (lib_id "Device:LED") (at 33.02 87.63 90) (unit 1)
     (in_bom yes) (on_board yes) (fields_autoplaced)
@@
       (reference "R2") (unit 1) (value "120") (footprint "Resistor_SMD:R_0603_1608Metric_Pad0.98x0.95mm_HandSolder")
     )
-    (path "/00000000-0000-0000-0000-00005c5151c5"
-      (reference "R4") (unit 1) (value "1k 7W") (footprint "Resistor_THT:R_Axial_Power_L25.0mm_W9.0mm_P30.48mm")
+    (path "/c008e4af-391b-4da0-80e9-6309dc522cc7"
+      (reference "R3") (unit 1) (value "500") (footprint "Package_TO_SOT_THT:TO-220-2_Horizontal_TabDown")
     )
     (path "/00000000-0000-0000-0000-00005c51b36b"
@@
       (reference "R6") (unit 1) (value "2k") (footprint "Resistor_SMD:R_0603_1608Metric")
     )
-    (path "/00000000-0000-0000-0000-00005ddba44f"
-      (reference "R7") (unit 1) (value "1k 7W") (footprint "Resistor_THT:R_Axial_Power_L25.0mm_W9.0mm_P30.48mm")
-    )
-  )
+  )

Commit message: Addded comments
Other:
- note added: "*NO Can New BMS"
- note added: "*Pack 2 negative to precharge"
- note added: "Batt -"
- note added: "Int +"
- note added: "Int -"
- note added: "Might be changed on footprint but is a copy of pac1"
- note added: "Same as pack #1 different layout"
Changed lines of the file:
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@@
+    (effects (font (size 1.27 1.27)) (justify left bottom))
+  )
+  (text "Int -\n" (at 42.545 24.13 0)
+    (effects (font (size 1.27 1.27) (thickness 0.254) bold italic) (justify left bottom))
+  )
+  (text "Batt -\n" (at 42.545 35.56 0)
+    (effects (font (size 1.27 1.27) (thickness 0.254) bold italic) (justify left bottom))
+  )
+  (text "Might be changed on footprint but is a copy of pac1"
+    (at 54.61 35.56 0)
+    (effects (font (size 1.27 1.27) bold italic) (justify left bottom))
+  )
+  (text "Same as pack #1 different layout" (at 215.265 179.705 0)
+    (effects (font (size 1.27 1.27) bold italic) (justify left bottom))
+  )
+  (text "*NO Can New BMS" (at 61.595 174.625 0)
     (effects (font (size 1.27 1.27)) (justify left bottom))
   )
@@
     (effects (font (size 1.27 1.27)) (justify left bottom))
   )
+  (text "*Pack 2 negative to precharge\n" (at 246.38 171.45 0)
+    (effects (font (size 1.27 1.27)) (justify left bottom))
+  )
   (text "39k, 3W resistor" (at 41.91 81.28 0)
     (effects (font (size 1.27 1.27)) (justify left bottom))
@@
     (effects (font (size 1.27 1.27)) (justify left bottom))
   )
+  (text "Int +\n" (at 42.545 46.99 0)
+    (effects (font (size 1.27 1.27) (thickness 0.254) bold italic) (justify left bottom))
+  )
   (text "Energy dissipated by 2 resistors when charging bus\ncapacitance (ONLY MOTOR CONTROLLER, FOR\nNOW): 20.7 Joules\n\nEnergy dissipated by 1 resistor: 20.7/2 Joules\n\nEquivalent pulse length: 0.25 seconds @ 288 Volts\n\nDatasheet specs 1000 Volt maximum for 0.25\nsecond pulse (so this resistor will work)"
